Commit message: Odom and Gmapping DONE(Map taken)

File: src/autobot_description/urdf/autobot.xacro (robot description, xacro)
@@ -4,5 +4,5 @@
      For more information, please see http://wiki.ros.org/sw_urdf_exporter -->
  <robot name="autobot" xmlns:xacro="http://www.ros.org/wiki/xacro">
- <xacro:include filename="$(find autobot)/urdf/autobot.gazebo" />
+ <xacro:include filename="$(find autobot_description)/urdf/autobot.gazebo" />
 <link name="base_footprint" />
   <link
@@ -28,5 +28,5 @@
       <geometry>
         <mesh
-          filename="package://autobot/meshes/base_link.STL" />
+          filename="package://autobot_description/meshes/base_link.STL" />
       </geometry>
       <material
@@ -42,5 +42,5 @@
       <geometry>
         <mesh
-          filename="package://autobot/meshes/base_link.STL" />
+          filename="package://autobot_description/meshes/base_link.STL" />
       </geometry>
     </collision>
@@ -72,5 +72,5 @@
       <geometry>
         <mesh
-          filename="package://autobot/meshes/lw_Link.STL" />
+          filename="package://autobot_description/meshes/lw_Link.STL" />
       </geometry>
       <material
@@ -86,5 +86,5 @@
       <geometry>
         <mesh
-          filename="package://autobot/meshes/lw_Link.STL" />
+          filename="package://autobot_description/meshes/lw_Link.STL" />
       </geometry>
     </collision>
@@ -125,5 +125,5 @@
       <geometry>
         <mesh
-          filename="package://autobot/meshes/rw_Link.STL" />
+          filename="package://autobot_description/meshes/rw_Link.STL" />
       </geometry>
       <material
@@ -139,5 +139,5 @@
       <geometry>
         <mesh
-          filename="package://autobot/meshes/rw_Link.STL" />
+          filename="package://autobot_description/meshes/rw_Link.STL" />
       </geometry>
     </collision>
@@ -178,5 +178,5 @@
       <geometry>
         <mesh
-          filename="package://autobot/meshes/sfw_Link.STL" />
+          filename="package://autobot_description/meshes/sfw_Link.STL" />
       </geometry>
       <material
@@ -192,5 +192,5 @@
       <geometry>
         <mesh
-          filename="package://autobot/meshes/sfw_Link.STL" />
+          filename="package://autobot_description/meshes/sfw_Link.STL" />
       </geometry>
     </collision>
@@ -231,5 +231,5 @@
       <geometry>
         <mesh
-          filename="package://autobot/meshes/sfw_Link.STL" />
+          filename="package://autobot_description/meshes/sfw_Link.STL" />
       </geometry>
       <material
@@ -245,5 +245,5 @@
       <geometry>
         <mesh
-          filename="package://autobot/meshes/sfw_Link.STL" />
+          filename="package://autobot_description/meshes/sfw_Link.STL" />
       </geometry>
     </collision>
@@ -266,5 +266,5 @@
     <inertial>
       <origin
-        xyz="0 0 -0.0203709532260616"
+        xyz="0 0 0"
         rpy="0 0 0" />
       <mass
@@ -284,5 +284,5 @@
       <geometry>
         <mesh
-          filename="package://autobot/meshes/laser.STL" />
+          filename="package://autobot_description/meshes/laser.STL" />
       </geometry>
       <material
@@ -298,5 +298,5 @@
       <geometry>
         <mesh
-          filename="package://autobot/meshes/laser.STL" />
+          filename="package://autobot_description/meshes/laser.STL" />
       </geometry>
     </collision>
@@ -306,6 +306,6 @@
     type="fixed">
     <origin
-      xyz="0.23948 -0.0026771 0.33"
-      rpy="0 0 3.14" />
+      xyz="0.18 0.21 0.40"
+      rpy="0 0 0" />
     <parent
       link="base_link" />
@@ -337,5 +337,5 @@
       <geometry>
         <mesh
-          filename="package://autobot/meshes/camera_Link.STL" />
+          filename="package://autobot_description/meshes/camera_Link.STL" />
       </geometry>
       <material
@@ -351,5 +351,5 @@
       <geometry>
         <mesh
-          filename="package://autobot/meshes/camera_Link.STL" />
+          filename="package://autobot_description/meshes/camera_Link.STL" />
       </geometry>
     </collision>
@@ -373,5 +373,5 @@
       <origin xyz="0 0 0" rpy="0 0 0"/>
       <geometry>
-        <mesh filename="package://autobot/meshes/imu.STL" />
+        <mesh filename="package://autobot_description/meshes/imu.STL" />
       </geometry>
     </collision>
@@ -379,5 +379,5 @@
       <origin xyz="0 0 0" rpy="0 0 0"/>
     <geometry>
-      <mesh filename="package://autobot/meshes/imu.STL" />
+      <mesh filename="package://autobot_description/meshes/imu.STL" />
       </geometry>
     </visual>
