Commit message: Modified URDF with intertial parameters

File: src/autobot_description/urdf/bot.xacro (robot description, xacro)
@@ -1,7 +1,24 @@
 <?xml version="1.0" ?>
 <robot name="autobot" xmlns:xacro="http://ros.org/wiki/xacro">
+<xacro:include filename="$(find autobot_description)/urdf/bot.gazebo" />
+<xacro:macro name="box_inertia" params="b_mass b_x b_y b_z">
+        <mass value="${b_mass}"/>
+        <inertia  ixx="${b_mass*(b_y*b_y+b_z*b_z)/12}" ixy = "0" ixz = "0"
+                  iyy="${b_mass*(b_x*b_x+b_z*b_z)/12}" iyz = "0"
+                  izz="${b_mass*(b_x*b_x+b_y*b_y)/12}"/>
+</xacro:macro>
+<xacro:macro name="cylinder_inertia" params="c_mass r l">
+        <mass value="${c_mass}"/>
+        <inertia  ixx="${c_mass*(3*r*r+l*l)/12}" ixy = "0" ixz = "0"
+                  iyy="${c_mass*(3*r*r+l*l)/12}" iyz = "0"
+                  izz="${c_mass*(r*r)/2}" />
+</xacro:macro>
 <link name="base_footprint" />
 <link name="base_link" >
-    <visual>
+  <inertial>
+    <origin xyz = "0 0 0" rpy = "0 0 0" />
+    <xacro:box_inertia b_mass="17" b_x = "0.72" b_y = "0.40" b_z = "0.28" />
+  </inertial>
+  <visual>
 	<origin xyz = "0 0 0" rpy = "0 0 0" />
         <geometry>
@@ -13,4 +30,5 @@
       </visual>
       <collision>
+        <origin xyz = "0 0 0" rpy = "0 0 0" />
         <geometry>
           <box size="0.72 0.40 0.28"/>
@@ -19,4 +37,9 @@
 </link>
 <link name="left_wheel" >
+ <origin xyz = "0 0 0" rpy = "0 0 0" />
+  <inertial>
+    <origin xyz = "0 0 0" rpy = "0 0 0" />
+    <xacro:cylinder_inertia c_mass = "2" r = "0.08" l = "0.06" />
+    </inertial>
   <visual>
     <origin xyz = "0 0 0" rpy = "0 0 0" />
@@ -29,4 +52,5 @@
   </visual>
   <collision>
+    <origin xyz = "0 0 0" rpy = "0 0 0" />
     <geometry>
       <cylinder length="0.06" radius="0.08"/>
@@ -35,6 +59,11 @@
 </link>
 <link name="right_wheel" >
+ <origin xyz = "0 0 0" rpy = "0 0 0" />
+  <inertial>
+    <origin xyz = "0 0 0" rpy = "0 0 0" />
+    <xacro:cylinder_inertia c_mass = "2" r = "0.08" l = "0.06" />
+    </inertial>
   <visual>
- <origin xyz = "0 0 0" rpy = "0 0 0" />
+    <origin xyz = "0 0 0" rpy = "0 0 0" />
     <geometry>
       <cylinder length="0.06" radius="0.08"/>
@@ -45,4 +74,5 @@
   </visual>
   <collision>
+    <origin xyz = "0 0 0" rpy = "0 0 0" />
     <geometry>
       <cylinder length="0.06" radius="0.08"/>
@@ -51,8 +81,13 @@
 </link>
 <link name="laser" >
-  <visual>
- <origin xyz = "0 0 0" rpy = "0 0 0" />
-      <geometry>
-        <box size="0.08 0.08 0.055"/>
+<origin xyz = "0 0 0" rpy = "0 0 0" />
+<inertial>
+  <mass value="0.09"/>
+      <inertia ixx="4.275e-05" ixy="0" ixz="0" iyy="4.275e-05" iyz="0" izz="5.5125e-05"/>
+</inertial>
+<visual>
+  <origin xyz = "0 0 0" rpy = "0 0 0" />
+       <geometry>
+        <cylinder length = "0.040" radius = "0.030" />
       </geometry>
       <material name="lidar_mat">
@@ -61,6 +96,7 @@
     </visual>
     <collision>
+      <origin xyz = "0 0 0" rpy = "0 0 0" />
       <geometry>
-        <box size="0.08 0.08 0.055"/>
+        <cylinder length = "0.040" radius = "0.030" />
       </geometry>
     </collision>

Commit message: Added model into AMR world

File: src/autobot_description/urdf/bot.xacro (robot description, xacro)
@@ -2,4 +2,5 @@
 <robot name="autobot" xmlns:xacro="http://ros.org/wiki/xacro">
 <xacro:include filename="$(find autobot_description)/urdf/bot.gazebo" />
+<xacro:include filename="$(find autobot_description)/urdf/bot.trans" />
 <xacro:macro name="box_inertia" params="b_mass b_x b_y b_z">
         <mass value="${b_mass}"/>
@@ -26,5 +27,5 @@
         </geometry>
         <material name="base_material">
-          <color rgba="1 1 1 1"/>
+          <color rgba="0 0 0 1"/>
         </material>
       </visual>
@@ -48,5 +49,5 @@
     </geometry>
     <material name="l_wheel">
-      <color rgba="1.5 0 2.5 1"/>
+      <color rgba="0 0 1 1"/>
     </material>
   </visual>
@@ -70,5 +71,5 @@
     </geometry>
     <material name="r_wheel">
-      <color rgba="1.5 0 2.5 1"/>
+      <color rgba="0 0 1 1"/>
     </material>
   </visual>
@@ -120,5 +121,5 @@
   <parent link = "base_link"/>
   <child link = "laser" />
-  <origin xyz = "0.18 0 0.18" rpy = "0 3.14 0" />
+  <origin xyz = "0.18 0 0.16" rpy = "0 3.14 0" />
 </joint>
 </robot>

Commit message: Added IMU and LiDAR Plugins to Robot

File: src/autobot_description/urdf/bot.xacro (robot description, xacro)
@@ -27,5 +27,5 @@
         </geometry>
         <material name="base_material">
-          <color rgba="0 0 0 1"/>
+          <color rgba="0 1 0 1"/>
         </material>
       </visual>
@@ -103,4 +103,33 @@
     </collision>
 </link>
+<!-- <link name = "front_castor" >
+  <origin xyz = "0 0 0" rpy = "0 0 0" />
+  <visual>
+    <origin xyz = "0 0 0" rpy = "0 0 0" />
+    <geometry>
+      <mesh filename="package://autobot_description/meshes/c_wheel.dae" />
+    </geometry>
+  </visual>
+</link> -->
+<!-- IMU -->
+  <link name="imu_link">
+    <collision>
+      <origin xyz="0 0 0" rpy="0 0 0"/>
+      <geometry>
+        <mesh filename="package://autobot_description/meshes/imu.STL" />
+      </geometry>
+    </collision>
+    <visual>
+      <origin xyz="0 0 0" rpy="0 0 0"/>
+    <geometry>
+      <mesh filename="package://autobot_description/meshes/imu.STL" />
+      </geometry>
+    </visual>
+    <inertial>
+      <mass value="1e-5" />
+      <origin xyz="0 0 0" rpy="0 0 0"/>
+      <inertia ixx="0" ixy="0" ixz="0" iyy="0" iyz="0" izz="0" />
+    </inertial>
+  </link>
 <joint name="footprint_link_joint" type="fixed" >
     <parent link = "base_footprint"/>
@@ -108,13 +137,15 @@
     <origin xyz = "0 0 0.20" rpy = "0 0 0" />
 </joint>
-<joint name="baselink_leftwheel" type="fixed" >
+<joint name="baselink_leftwheel" type="continuous" >
+  <axis xyz = "0 0 1" />
   <parent link = "base_link"/>
   <child link = "left_wheel" />
-  <origin xyz = "0 0.23 -0.12" rpy = "1.57 0 0" />
+  <origin xyz = "0 0.23 -0.12" rpy = "1.57 0 3.14 " />
 </joint>
-<joint name="baselink_rightwheel" type="fixed" >
+<joint name="baselink_rightwheel" type="continuous" >
+  <axis xyz = "0 0 1" />
   <parent link = "base_link"/>
   <child link = "right_wheel" />
-  <origin xyz = "0 -0.23 -0.12" rpy = "1.57 0 0" />
+  <origin xyz = "0 -0.23 -0.12" rpy = "1.57 0 3.14" />
 </joint>
 <joint name="baselink_lidar" type="fixed" >
@@ -123,3 +154,9 @@
   <origin xyz = "0.18 0 0.16" rpy = "0 3.14 0" />
 </joint>
+<joint name="imujoint" type="fixed">
+    <origin xyz="0.132 0.26 0.36" rpy="0 0 0" />
+    <parent link="base_link" />
+    <child link="imu_link" />
+    <axis xyz="0 0 0" />
+</joint>
 </robot>

Commit message: Modified URDF for IMU Scale

File: src/autobot_description/urdf/bot.xacro (robot description, xacro)
@@ -117,5 +117,5 @@
       <origin xyz="0 0 0" rpy="0 0 0"/>
       <geometry>
-        <mesh filename="package://autobot_description/meshes/imu.STL" />
+        <mesh filename="package://autobot_description/meshes/imu.STL" scale= "0.001 0.001 0.001"/>
       </geometry>
     </collision>
@@ -123,5 +123,5 @@
       <origin xyz="0 0 0" rpy="0 0 0"/>
     <geometry>
-      <mesh filename="package://autobot_description/meshes/imu.STL" />
+      <mesh filename="package://autobot_description/meshes/imu.STL" scale="0.001 0.001 0.001"/>
       </geometry>
     </visual>
@@ -155,5 +155,5 @@
 </joint>
 <joint name="imujoint" type="fixed">
-    <origin xyz="0.132 0.26 0.36" rpy="0 0 0" />
+    <origin xyz="0 0 0" rpy="0 0 0" />
     <parent link="base_link" />
     <child link="imu_link" />

Commit message: Added Castor wheel to bot

File: src/autobot_description/urdf/bot.xacro (robot description, xacro)
@@ -103,13 +103,42 @@
     </collision>
 </link>
-<!-- <link name = "front_castor" >
-  <origin xyz = "0 0 0" rpy = "0 0 0" />
-  <visual>
-    <origin xyz = "0 0 0" rpy = "0 0 0" />
-    <geometry>
-      <mesh filename="package://autobot_description/meshes/c_wheel.dae" />
-    </geometry>
-  </visual>
-</link> -->
+<link name="frontCastor_link">
+  <collision>
+    <origin xyz="0 0 0" rpy="0 0 0"/>
+    <geometry>
+      <mesh filename="package://autobot_description/meshes/castor_wheel.STL" scale= "0.001 0.001 0.001"/>
+    </geometry>
+  </collision>
+  <visual>
+    <origin xyz="0 0 0" rpy="0 0 0"/>
+  <geometry>
+    <mesh filename="package://autobot_description/meshes/castor_wheel.STL" scale="0.001 0.001 0.001"/>
+    </geometry>
+  </visual>
+  <inertial>
+    <mass value="0.30" />
+    <origin xyz="0 0 0" rpy="0 0 0"/>
+    <inertia ixx="0" ixy="0" ixz="0" iyy="0" iyz="0" izz="0" />
+  </inertial>
+</link>
+<link name="backCastor_link">
+  <collision>
+    <origin xyz="0 0 0" rpy="0 0 0"/>
+    <geometry>
+      <mesh filename="package://autobot_description/meshes/castor_wheel.STL" scale= "0.001 0.001 0.001"/>
+    </geometry>
+  </collision>
+  <visual>
+    <origin xyz="0 0 0" rpy="0 0 0"/>
+  <geometry>
+    <mesh filename="package://autobot_description/meshes/castor_wheel.STL" scale="0.001 0.001 0.001"/>
+    </geometry>
+  </visual>
+  <inertial>
+    <mass value="0.30" />
+    <origin xyz="0 0 0" rpy="0 0 0"/>
+    <inertia ixx="0" ixy="0" ixz="0" iyy="0" iyz="0" izz="0" />
+  </inertial>
+</link>
 <!-- IMU -->
   <link name="imu_link">
@@ -155,8 +184,18 @@
 </joint>
 <joint name="imujoint" type="fixed">
-    <origin xyz="0 0 0" rpy="0 0 0" />
+    <origin xyz="0.228 -0.008 0" rpy="1.57 0 1.57" />
     <parent link="base_link" />
     <child link="imu_link" />
     <axis xyz="0 0 0" />
 </joint>
+<joint name="frontCastor_joint" type="continuous" >
+    <origin xyz = "0.30 0 -0.14" rpy = "0 0 0" />
+    <parent link="base_link" />
+    <child link ="frontCastor_link" />
+</joint>
+<joint name="backCastor_joint" type="continuous" >
+  <origin xyz = "-0.30 0 -0.14" rpy = "0 0 0" />
+  <parent link="base_link" />
+  <child link ="backCastor_link" />
+</joint>
 </robot>

Commit message: modified urdf

File: src/autobot_description/urdf/bot.xacro (robot description, xacro)
@@ -119,5 +119,5 @@
     <mass value="0.30" />
     <origin xyz="0 0 0" rpy="0 0 0"/>
-    <inertia ixx="0" ixy="0" ixz="0" iyy="0" iyz="0" izz="0" />
+    <inertia ixx="0.0144" ixy="0" ixz="0" iyy="0.0144" iyz="0" izz="0.0144" />
   </inertial>
 </link>
@@ -138,5 +138,5 @@
     <mass value="0.30" />
     <origin xyz="0 0 0" rpy="0 0 0"/>
-    <inertia ixx="0" ixy="0" ixz="0" iyy="0" iyz="0" izz="0" />
+    <inertia ixx="0.0144" ixy="0" ixz="0" iyy="0.0144" iyz="0" izz="0.0144" />
   </inertial>
 </link>
@@ -189,10 +189,10 @@
     <axis xyz="0 0 0" />
 </joint>
-<joint name="frontCastor_joint" type="continuous" >
+<joint name="frontCastor_joint" type="fixed" >
     <origin xyz = "0.30 0 -0.14" rpy = "0 0 0" />
     <parent link="base_link" />
     <child link ="frontCastor_link" />
 </joint>
-<joint name="backCastor_joint" type="continuous" >
+<joint name="backCastor_joint" type="fixed" >
   <origin xyz = "-0.30 0 -0.14" rpy = "0 0 0" />
   <parent link="base_link" />

Commit message: Added a short area map and checked AMCL - Yas

File: src/autobot_description/urdf/bot.xacro (robot description, xacro)
@@ -180,5 +180,5 @@
   <parent link = "base_link"/>
   <child link = "laser" />
-  <origin xyz = "0.18 0 0.16" rpy = "0 3.14 0" />
+  <origin xyz = "0.18 0 0.16" rpy = "3.14 3.14 0" />
 </joint>
 <joint name="imujoint" type="fixed">

Commit message: Modified IMU position

File: src/autobot_description/urdf/bot.xacro (robot description, xacro)
@@ -20,5 +20,5 @@
     <xacro:box_inertia b_mass="17" b_x = "0.72" b_y = "0.40" b_z = "0.28" />
   </inertial>
-  <visual>
+  <!-- <visual>
 	<origin xyz = "0 0 0" rpy = "0 0 0" />
         <geometry>
@@ -28,5 +28,5 @@
           <color rgba="0 1 0 1"/>
         </material>
-      </visual>
+      </visual> -->
       <collision>
         <origin xyz = "0 0 0" rpy = "0 0 0" />
@@ -183,5 +183,5 @@
 </joint>
 <joint name="imujoint" type="fixed">
-    <origin xyz="0.228 -0.008 0" rpy="1.57 0 1.57" />
+    <origin xyz="0.216 0 0.116" rpy="1.57 0 1.57" />
     <parent link="base_link" />
     <child link="imu_link" />

Commit message: Added imu

File: src/autobot_description/urdf/bot.xacro (robot description, xacro)
@@ -180,5 +180,5 @@
   <parent link = "base_link"/>
   <child link = "laser" />
-  <origin xyz = "0.18 0 0.16" rpy = "3.14 3.14 0" />
+  <origin xyz = "0.18 0 0.16" rpy = "0 3.14 0" />
 </joint>
 <joint name="imujoint" type="fixed">

Commit message: modified amcl and navigation stack params

File: src/autobot_description/urdf/bot.xacro (robot description, xacro)
@@ -20,5 +20,5 @@
     <xacro:box_inertia b_mass="17" b_x = "0.72" b_y = "0.40" b_z = "0.28" />
   </inertial>
-  <!-- <visual>
+  <visual>
 	<origin xyz = "0 0 0" rpy = "0 0 0" />
         <geometry>
@@ -28,5 +28,5 @@
           <color rgba="0 1 0 1"/>
         </material>
-      </visual> -->
+      </visual>
       <collision>
         <origin xyz = "0 0 0" rpy = "0 0 0" />

Commit message: Added Cameras to robot model, Edit in Footprint size

File: src/autobot_description/urdf/bot.xacro (robot description, xacro)
@@ -160,4 +160,44 @@
     </inertial>
   </link>
+  <!-- Camera T265 link -->
+    <link name="t265_link">
+    <collision>
+      <origin xyz="0 0 0" rpy="0 0 0"/>
+      <geometry>
+        <mesh filename="package://autobot_description/meshes/T265.STL" scale="0.001 0.001 0.001"/>
+      </geometry>
+    </collision>
+    <visual>
+      <origin xyz="0 0 0" rpy="0 0 0"/>
+    <geometry>
+      <mesh filename="package://autobot_description/meshes/T265.STL" scale="0.001 0.001 0.001"/>
+      </geometry>
+    </visual>
+    <inertial>
+      <mass value="1e-5" />
+      <origin xyz="0 0 0" rpy="0 0 0"/>
+      <inertia ixx="0" ixy="0" ixz="0" iyy="0" iyz="0" izz="0" />
+    </inertial>
+  </link>
+  <!-- Camera D435i link -->
+    <link name="d435_link">
+    <collision>
+      <origin xyz="0 0 0" rpy="0 0 0"/>
+      <geometry>
+        <mesh filename="package://autobot_description/meshes/D435i.STL" scale="0.001 0.001 0.001"/>
+      </geometry>
+    </collision>
+    <visual>
+      <origin xyz="0 0 0" rpy="0 0 0"/>
+    <geometry>
+      <mesh filename="package://autobot_description/meshes/D435i.STL" scale="0.001 0.001 0.001"/>
+      </geometry>
+    </visual>
+    <inertial>
+      <mass value="1e-5" />
+      <origin xyz="0 0 0" rpy="0 0 0"/>
+      <inertia ixx="0" ixy="0" ixz="0" iyy="0" iyz="0" izz="0" />
+    </inertial>
+  </link>
 <joint name="footprint_link_joint" type="fixed" >
     <parent link = "base_footprint"/>
@@ -198,3 +238,13 @@
   <child link ="backCastor_link" />
 </joint>
+<joint name="t265_joint" type="fixed" >
+  <origin xyz = "0.425 0 -0.12" rpy = "1.57 0 -1.57" />
+  <parent link="base_link" />
+  <child link ="t265_link" />
+</joint>
+<joint name="d435_joint" type="fixed" >
+  <origin xyz = "0.395 0 -0.065" rpy = "1.57 0 -1.57" />
+  <parent link="base_link" />
+  <child link ="d435_link" />
+</joint>
 </robot>

Commit message: final changes-01

File: src/autobot_description/urdf/bot.xacro (robot description, xacro)
@@ -220,5 +220,5 @@
   <parent link = "base_link"/>
   <child link = "laser" />
-  <origin xyz = "0.18 0 0.16" rpy = "3.14 3.14 0" />
+  <origin xyz = "0.18 0 0.16" rpy = "0 3.14 0" />
 </joint>
 <joint name="imujoint" type="fixed">

Commit message: Added pointcloud to laserscan node in simulation - Tuning pending for DWA

File: src/autobot_description/urdf/bot.xacro (robot description, xacro)
@@ -189,5 +189,5 @@
     </collision>
     <visual>
-      <origin xyz="0 0 0" rpy="0 0 0"/>
+      <origin xyz="0 0 0" rpy="1.57 0 1.57"/>
     <geometry>
       <mesh filename="package://autobot_description/meshes/D435i.STL" scale="0.001 0.001 0.001"/>
@@ -200,4 +200,5 @@
     </inertial>
   </link>
+<link name="camera_depth" />
 <joint name="footprint_link_joint" type="fixed" >
     <parent link = "base_footprint"/>
@@ -244,7 +245,12 @@
 </joint>
 <joint name="d435_joint" type="fixed" >
-  <origin xyz = "0.395 0 -0.065" rpy = "1.57 0 -1.57" />
+  <origin xyz = "0.395 0 -0.065" rpy = "0 0 0" />
   <parent link="base_link" />
   <child link ="d435_link" />
 </joint>
+<joint name="depth_joint" type="fixed" >
+  <origin xyz = "0.395 0 -0.065" rpy = "-1.57 0 -1.57" />
+  <parent link="base_link" />
+  <child link ="camera_depth" />
+</joint>
 </robot>

Commit message: Edit for bot.xacro

File: src/autobot_description/urdf/bot.xacro (robot description, xacro)
@@ -220,11 +220,11 @@
   <parent link = "base_link"/>
   <child link = "laser" />
-  <origin xyz = "0.18 0 0.16" rpy = "0 3.14 0" />
+  <origin xyz = "0.18 0 0.16" rpy = "3.14 3.14 0" />
 </joint>
 <joint name="imujoint" type="fixed">
-    <origin xyz="0.216 0 0.116" rpy="1.57 0 1.57" />
+    <origin xyz="0.216 0 0.216" rpy="3.14 3.14 0" />
     <parent link="base_link" />
     <child link="imu_link" />
-    <axis xyz="0 0 0" />
+    <axis xyz="0 0 1" />
 </joint>
 <joint name="frontCastor_joint" type="fixed" >

Commit message: small changes in costmap params

File: src/autobot_description/urdf/bot.xacro (robot description, xacro)
@@ -181,5 +181,5 @@
   </link>
   <!-- Camera D435i link -->
-    <link name="d435_link">
+    <link name="camera_link">
     <collision>
       <origin xyz="0 0 0" rpy="0 0 0"/>
@@ -247,5 +247,5 @@
   <origin xyz = "0.395 0 -0.065" rpy = "0 0 0" />
   <parent link="base_link" />
-  <child link ="d435_link" />
+  <child link ="camera_link" />
 </joint>
 <joint name="depth_joint" type="fixed" >

Commit message: Final changes Commit

File: src/autobot_description/urdf/bot.xacro (robot description, xacro)
@@ -149,5 +149,5 @@
     </collision>
     <visual>
-      <origin xyz="0 0 0" rpy="0 0 0"/>
+      <origin xyz="0 0 0" rpy="1.57 0 1.57"/>
     <geometry>
       <mesh filename="package://autobot_description/meshes/imu.STL" scale="0.001 0.001 0.001"/>
